Commit message: lift up lidar to avoid from sensing each other

File: src/turtlebot3/turtlebot3_description/urdf/turtlebot3_burger.urdf.xacro (robot description, xacro)
@@ -116,5 +116,5 @@
     <parent link="$(arg robotName)_base_link"/>
     <child link="$(arg robotName)_base_scan"/>
-    <origin xyz="-0.032 0 0.172" rpy="0 0 0"/>
+    <origin xyz="-0.032 0 0.202" rpy="0 0 0"/>
   </joint>
   <link name="$(arg robotName)_base_scan">
@@ -126,10 +126,10 @@
       <material name="dark"/>
     </visual>
-    <collision>
+    <!-- <collision>
       <origin xyz="0.015 0 -0.0065" rpy="0 0 0"/>
       <geometry>
         <cylinder length="0.0315" radius="0.055"/>
       </geometry>
-    </collision>
+    </collision> -->
     <inertial>
       <mass value="0.114" />
